Commit message: Added: Forgot to add revolute joints to some joints in tbot_left_arm

File: talos_navigation/urdf/tbot_left_arm.urdf.xacro (robot description, xacro)
@@ -36,5 +36,5 @@
 	</visual>
 </link>
-<joint name="body_to_left_shoulder" type="fixed">
+<joint name="body_to_left_shoulder" type="revolute">
 	<!-- Note: Crude approximation of physical robot -->
   	<parent link="body"/>
@@ -85,5 +85,5 @@
 	</visual>
 </link>
-<joint name="shoulder_to_upper_arm" type="fixed">
+<joint name="shoulder_to_upper_arm" type="revolute">
         <!-- Note: Crude approximation of the joint, this is not the exact connecting joint location -->
   	<parent link="left_shoulder"/>
