Commit message: Added: Complete torso .urdf.xacro that is ready (except for the TODOs) for integration with talos_common.urdf.xacro

File: talos_navigation/talos_description/urdf/torso_v0/talos_torso.urdf.xacro (robot description, xacro)
@@ -11,5 +11,73 @@
   <xacro:include filename="$(find pr2_description)/urdf/sensors/microstrain_3dmgx2_imu.urdf.xacro" />
 -->
+<!--                                               -->
+<!--                 TORSO CONSTANTS               -->
+<!--                                               -->
+<!-- TODO: Set proper values for the torso efforts and vels -->
+<property name="max_torso_effort" value="10" />
+<property name="max_torso_velocity" value="10" />
+<property name="torso_friction" value="0" />
+<property name="torso_damping" value="0" />
+<property name="max_torso_velocity" value="10" />
+<property name="torso_safety_k_velocity" value="10"/>
+<property name="torso_mass" value="10" />
+<!--                                               -->
+<!--                TORSO DEFINITION               -->
+<!--                                               -->
 <xacro:macro name="talos_torso" params="name parent *origin">
+<joint name="${name}_rotating_joint" type="continuous">
+	<axis xyz="0 0 1" />
+	<parent link="${parent}"/>
+	<child link="${name}_link"/>
+	<origin rpy="0 0 0" xyz="0 0 0"/>
+       <!-- TODO: Set appropriate values for these -->
+	<limit effort="${max_torso_effort}" velocity="${max_wheel_velocity}"/> <!-- alpha tested effort and velocity limits -->
+       <!-- TODO: Set appropriate values for these -->
+	<safety_controller k_velocity="${safety_k_velocity}" />
+	<dynamics damping="${torso_damping}" friction="${torso_friction}" />
+</joint>
+<link name="${name}_link">
+<!-- TODO: Set appropriate values for these -->
+<!--
+ <inertial>
+        <mass value="${torso_mass}" />
+        <origin xyz="-0.1 0 -0.0885" />
+        <inertia ixx="2.771653750257" ixy="0.004284522609" ixz="-0.160418504506"
+                 iyy="2.510019507959" iyz="0.029664468704" izz="0.526432355569" />
+      </inertial>
+-->
+      <visual>
+        <origin xyz="0 0 0" rpy="0 0 0" />
+	 <!-- TODO: Add the correct .dae path for geometry -->
+        <!-- <geometry>
+          <mesh filename="package://pr2_description/meshes/torso_v0/torso_lift.dae" />
+        </geometry>
+	 -->
+	<!-- Temporary, because we will be using the .dae -->
+	<geometry>
+		<box size="0.4 0.4 1.0"/>
+	</geometry>
+	<material name="white">
+		<color rgba="1 1 1 1"/>
+	</material>
+	</visual>
+	<!-- TODO: Add collision .stl file
+	<collision name="${name}_collision">
+        <origin xyz="0 0 0" rpy="0 0 0" />
+        <geometry>
+          <mesh filename="package://pr2_description/meshes/torso_v0/torso_lift_L.stl" />
+        </geometry>
+      </collision>
+	-->
+</link>
+<!-- TODO: Add proper extensions for simulator and transmissions
+    <xacro:pr2_torso_gazebo_v0 name="${name}" />
+    <xacro:pr2_torso_transmission_v0 name="${name}" />
+-->
+<!-- TODO: Possibly add an IMU? The PR2 has one and I'm not sure if we have one or not
+    <xacro:microstrain_3dmgx2_imu_v0 name="imu" parent="${name}" imu_topic="torso_lift_imu/data" update_rate="100.0" stdev="0.00017" >
+        <origin xyz="-0.02977 -0.1497 0.164" rpy="0 ${M_PI} 0" />
+    </xacro:microstrain_3dmgx2_imu_v0>
+-->
 </xacro:macro>
 </robot>
