Commit message: Added: Refactored arm into xacro for proper design

File: talos_navigation/talos_description/urdf/upper_arm_v0/tbot_upper_arm_v0.urdf.xacro (robot description, xacro)
@@ -7,7 +7,6 @@
   <xacro:include filename="$(find pr2_description)/urdf/upper_arm_v0/upper_arm.transmission.xacro" />
   <xacro:include filename="$(find pr2_description)/urdf/common.xacro" /> -->
+<!-- BELOW IS DEPRECATED
 <link name="left_shoulder">
-	<!-- TODO: Jordan start -->
-	<!-- TODO Jordan: Please fill in the required values specified by "0" or near approximations -->
 	<inertial>
 		<mass value="0" />
@@ -17,10 +16,7 @@
 			  izz="0" />
 	</inertial>
-        <!-- TODO: Jordan end -->
-        <!-- TODO: Someone? Not sure how these are done yet. -->
 	<collision>
 		<origin xyz="0 0 0" rpy="0 0 0" />
 		<geometry>
-		  <!-- <mesh filename="package://pr2_description/meshes/upper_arm_v0/elbow_flex.stl" /> -->
 		</geometry>
 	</collision>
@@ -30,5 +26,4 @@
 		</geometry>
 		<origin rpy="0 0 0" xyz="0 0 0"/>
-		<!-- TODO: Add meshes -->
 		<material name="white">
 			<color rgba="1 1 1 1"/>
@@ -37,23 +32,13 @@
 </link>
 <joint name="body_to_left_shoulder" type="revolute">
-	<!-- Note: Crude approximation of physical robot -->
   	<parent link="body"/>
 	<child link="left_shoulder"/>
 	<origin rpy="0 0 1.57" xyz="-0.25 -0.1 -0.39"/>
- 	<!-- TODO Jordan Start: -->
-        <!-- TODO Jordan: Please fill in the required values specified by "?" or near approximations -->
-	<!-- Note: Code template taken from PR2_upper_arm.urdf for templating -->
-	<!-- Doc: axis of revolution -->
 	<axis xyz="0 1 0" />
-	<!-- TODO Jordan: lower rotation degree w.r.t specified axis, same thing for upper. Effort is max force in newtons. Velocity is max velocity of joint. -->
 	<limit lower="?" upper="?" effort="?" velocity="${VELOCITY_LIMIT_SCALE*5.5}" />
-        <!-- Note: PR2 Has safety controller, not sure what it's for yet or what the values do-->
-	<!-- <safety_controller k_position="100" k_velocity="3" soft_lower_limit="${-2.3213+0.2}" soft_upper_limit="${0.00-0.15}" /> -->
-        <!-- Note: Jordan, do you know what this could be? -->
 	<calibration falling="${-1.1606 + cal_r_elbow_flex_flag}"/>
-        <!-- TODO: Jordan do you know what goes here? I'm not sure-->
 	<dynamics damping="?" />
-        <!-- TODO: Jordan end: -->
 </joint>
+ ABOVE IS DEPRECATED -->
 <link name="left_upper_arm">
 	<!-- TODO: Jordan start -->
