Commit message: Added: Proper naming for talos arm

File: talos_navigation/talos_description/urdf/upper_arm_v0/talos_upper_arm_v1.urdf.xacro (robot description, xacro)
@@ -31,5 +31,5 @@
 <property name="shoulder_joint_calibration_falling" value="0" />
 <property name="shoulder_joint_damping" value="0" />
-<xacro:macro name="talos_shoulder" params="side parent reflect">
+<xacro:macro name="talos_upper_arm" params="side parent reflect">
 <joint name="${side}_shoulder_joint" type="fixed">
 	<!-- TODO: Add proper values for xyz -->
