Commit message: Added: Made changes to stacked DAE that I forgot to add to commit Added: Modifed talos_base to reflect upcoming deprecations

File: talos_navigation/talos_description/urdf/talos_common.xacro (robot description, xacro)
@@ -2,5 +2,5 @@
 <robot xmlns:xacro="http://www.ros.org/wiki/xacro" name="talos">
   <!-- Base Plate and Spokes -->
-<!-- TODO: Add meshes -->
+<!-- Refactored already to the new .urdf.xacro, this code until ending specified is DEPRECATED
   <link name="horizontal_base_plate">
   	<visual>
@@ -14,5 +14,4 @@
 	</visual>
   </link>
-<!-- TODO: Add meshes -->
   <joint name="base_plate_to_base_bar" type="fixed">
   	<parent link="horizontal_base_plate"/>
@@ -20,5 +19,4 @@
 	<origin xyz="0.1 0 0" rpy="0 0 0"/>
   </joint>
-<!-- TODO: Add meshes -->
   <link name="horizontal_base_plate_bar">
     <visual>
@@ -32,5 +30,4 @@
     </visual>
   </link>
-<!-- TODO: Add meshes -->
   <link name="lwheel_spoke">
 	<visual>
@@ -44,5 +41,4 @@
 	</visual>
   </link>
-<!-- TODO: Add meshes -->
   <link name="rwheel_spoke">
 	<visual>
@@ -56,5 +52,4 @@
 	</visual>
   </link>
-<!-- TODO: Add meshes -->
   <joint name="base_plate_to_lwheel_spoke" type="fixed">
 	<parent link="horizontal_base_plate"/>
@@ -62,12 +57,9 @@
 	<origin rpy="1.57 0 0" xyz="0 -0.235 0"/>
   </joint>
-<!-- TODO: Add meshes -->
-  <joint name="base_plate_to_rwheel_spoke" type="fixed">
+<joint name="base_plate_to_rwheel_spoke" type="fixed">
 	<parent link="horizontal_base_plate"/>
 	<child link="rwheel_spoke"/>
 	<origin rpy="1.57 0 0" xyz="0 0.235 0"/>
-  </joint>
-										<!-- Wheels -->
-<!-- TODO: Add meshes -->
+</joint>
   <link name="lwheel">
 	<visual>
@@ -81,5 +73,4 @@
 	</visual>
   </link>
-<!-- TODO: Add meshes -->
   <link name="rwheel">
 	<visual>
@@ -93,5 +84,4 @@
 	</visual>
   </link>
-<!-- TODO: Add meshes -->
   <joint name="lwheel_spoke_to_lwheel" type="fixed">
 	<parent link="lwheel_spoke"/>
@@ -99,5 +89,4 @@
 	<origin rpy="0 0 0" xyz="0 0 0.04"/>
   </joint>
-<!-- TODO: Add meshes -->
   <joint name="rwheel_spoke_to_rwheel" type="fixed">
 	<parent link="rwheel_spoke"/>
@@ -105,6 +94,4 @@
 	<origin rpy="0 0 0" xyz="0 0 -0.04"/>
   </joint>
-									<!-- Aluminum Frame -->
-<!-- TODO: Add meshes -->
   <link name="lwheel_bottom_bar">
 	<visual>
@@ -118,5 +105,4 @@
     </visual>
   </link>
-<!-- TODO: Add meshes -->
  <link name="rwheel_bottom_bar">
 	<visual>
@@ -130,5 +116,4 @@
     </visual>
   </link>
-<!-- TODO: Add meshes -->
  <joint name="base_plate_bar_to_lwheel_bottom_bar" type="fixed">
 	<parent link="horizontal_base_plate_bar"/>
@@ -136,5 +121,4 @@
 	<origin rpy="0 0 1.57" xyz="-0.295 -0.31 0"/>
   </joint>
-<!-- TODO: Add meshes -->
  <joint name="base_plate_bar_to_rwheel_bottom_bar" type="fixed">
 	<parent link="horizontal_base_plate_bar"/>
@@ -142,5 +126,4 @@
 	<origin rpy="0 0 1.57" xyz="-0.295 0.31 0"/>
   </joint>
-<!-- TODO: Add meshes -->
   <link name="bottom_bar_opposite_from_wheels">
 	<visual>
@@ -154,5 +137,4 @@
     </visual>
   </link>
-<!-- TODO: Add meshes -->
   <joint name="rwheel_bottom_bar_to_opposite_bottom_bar" type="fixed">
 	<parent link="rwheel_bottom_bar"/>
@@ -160,5 +142,4 @@
 	<origin rpy="0 0 1.57" xyz="-0.295 0.295 0"/>
   </joint>
-<!-- TODO: Add meshes -->
   <joint name="lwheel_bottom_bar_to_opposite_bottom_bar" type="fixed">
   	<parent link="lwheel_bottom_bar"/>
@@ -166,5 +147,4 @@
 	<origin rpy="0 0 0" xyz="0 0 0"/>
   </joint>
-<!-- TODO: Add meshes -->
   <link name="opposite_vertical_rwheel_bar">
 	<visual>
@@ -178,5 +158,4 @@
     </visual>
   </link>
-<!-- TODO: Add meshes -->
   <joint name="rwheel_bottom_bar_to_ov_rwheel_bar" type="fixed">
   	<parent link="rwheel_bottom_bar"/>
@@ -184,5 +163,4 @@
 	<origin rpy="1.57 0 0" xyz="0 0.295 0.16438"/>
   </joint>
-<!-- TODO: Add meshes -->
   <link name="opposite_vertical_lwheel_bar">
 	<visual>
@@ -196,5 +174,4 @@
     </visual>
   </link>
-<!-- TODO: Add meshes -->
 <joint name="lwheel_bottom_bar_to_ov_lwheel_bar" type="fixed">
   	<parent link="lwheel_bottom_bar"/>
@@ -202,5 +179,4 @@
 	<origin rpy="1.57 0 0" xyz="0 0.295 0.16438"/>
   </joint>
-<!-- TODO: Add meshes -->
 <link name="vertical_lwheel_bar">
 	<visual>
@@ -214,5 +190,4 @@
     </visual>
   </link>
-<!-- TODO: Add meshes -->
 <joint name="lwheel_bottom_bar_to_v_lwheel_bar" type="fixed">
   	<parent link="lwheel_bottom_bar"/>
@@ -220,5 +195,4 @@
 	<origin rpy="1.57 0 0" xyz="0 -0.295 0.16438"/>
   </joint>
-<!-- TODO: Add meshes -->
 <link name="vertical_rwheel_bar">
 	<visual>
@@ -232,5 +206,4 @@
     </visual>
   </link>
-<!-- TODO: Add meshes -->
 <joint name="lwheel_bottom_bar_to_v_rwheel_bar" type="fixed">
   	<parent link="rwheel_bottom_bar"/>
@@ -238,5 +211,4 @@
 	<origin rpy="1.57 0 0" xyz="0 -0.295 0.16438"/>
   </joint>
-<!-- TODO: Add meshes -->
 <link name="top_plate">
 	<visual>
@@ -250,5 +222,4 @@
     </visual>
   </link>
-<!-- TODO: Add meshes -->
 <joint name="v_rwheel_bar_to_top_plate" type="fixed">
   	<parent link="vertical_rwheel_bar"/>
@@ -256,5 +227,4 @@
 	<origin rpy="1.57 0 0" xyz="-0.31 0.16438 -0.294525"/>
   </joint>
-<!-- TODO: Add meshes -->
 <joint name="v_lwheel_bar_to_top_plate" type="fixed">
   	<parent link="vertical_lwheel_bar"/>
@@ -262,5 +232,4 @@
 	<origin rpy="0 0 0" xyz="0 0 0"/>
   </joint>
-<!-- TODO: Add meshes -->
 <joint name="opposite__vertical_lwheel_bar_to_top_plate" type="fixed">
   	<parent link="opposite_vertical_lwheel_bar"/>
@@ -268,5 +237,4 @@
 	<origin rpy="0 0 0" xyz="0 0 0"/>
   </joint>
-<!-- TODO: Add meshes -->
 <joint name="opposite__vertical_rwheel_bar_to_top_plate" type="fixed">
   	<parent link="opposite_vertical_rwheel_bar"/>
@@ -274,5 +242,4 @@
 	<origin rpy="0 0 0" xyz="0 0 0"/>
   </joint>
-<!-- TODO: Add meshes -->
 <link name="right_castor_spoke">
 	<visual>
@@ -286,5 +253,4 @@
 	</visual>
   </link>
-<!-- TODO: Add meshes -->
 <link name="left_castor_spoke">
 	<visual>
@@ -298,5 +264,4 @@
 	</visual>
   </link>
-<!-- TODO: Add meshes -->
 <joint name="rwheel_bottom_bar_to_rwheel_castor_spoke" type="fixed">
   	<parent link="rwheel_bottom_bar"/>
@@ -304,5 +269,4 @@
 	<origin rpy="0 1.57 0" xyz="-0.035 0.2 0"/>
   </joint>
-<!-- TODO: Add meshes -->
 <joint name="lwheel_bottom_bar_to_lwheel_castor_spoke" type="fixed">
   	<parent link="lwheel_bottom_bar"/>
@@ -310,5 +274,4 @@
 	<origin rpy="0 1.57 0" xyz="0.035 0.2 0"/>
   </joint>
-<!-- TODO: Add meshes -->
 <link name="right_castor_wheel">
 	<visual>
@@ -322,5 +285,4 @@
 	</visual>
   </link>
-<!-- TODO: Add meshes -->
 <link name="left_castor_wheel">
 	<visual>
@@ -334,5 +296,4 @@
 	</visual>
   </link>
-<!-- TODO: Add meshes -->
 <joint name="right_castor_spoke_to_right_castor_wheel" type="fixed">
   	<parent link="right_castor_spoke"/>
@@ -340,5 +301,4 @@
 	<origin rpy="0 0 0" xyz="0 0 -0.03805"/>
   </joint>
-<!-- TODO: Add meshes -->
 <joint name="left_castor_spoke_to_left_castor_wheel" type="fixed">
   	<parent link="left_castor_spoke"/>
@@ -346,6 +306,4 @@
 	<origin rpy="0 0 0" xyz="0 0 0.03805"/>
   </joint>
-<!-- Rotational Base -->
-<!-- TODO: Add meshes -->
 <link name="rotational_base_plate">
 	<visual>
@@ -359,5 +317,4 @@
 	</visual>
   </link>
-<!-- TODO: Add meshes -->
 <joint name="top_plate_to_rotational_base" type="fixed">
   	<parent link="top_plate"/>
@@ -365,5 +322,4 @@
 	<origin rpy="0 0 0" xyz="0 0 -0.015"/>
 </joint>
-<!-- TODO: Add meshes -->
 <link name="top_rotating_plate">
 	<visual>
@@ -377,12 +333,9 @@
 	</visual>
   </link>
-<!-- TODO: Add meshes -->
 <joint name="rotational_base_connection" type="fixed">
   	<parent link="rotational_base_plate"/>
 	<child link="top_rotating_plate"/>
 	<origin rpy="0 0 0" xyz="0 0 0"/>
- 	<!-- <limit effort="30" velocity="1.0" lower="1.5" upper="1.5"/> -->
-</joint>
-<!-- TODO: Add meshes -->
+</joint>
   <link name="body">
 	<visual>
@@ -396,5 +349,4 @@
     </visual>
   </link>
-<!-- TODO: Add meshes -->
 <joint name="top_rotating_plate_to_body" type="fixed">
   	<parent link="top_rotating_plate"/>
@@ -402,4 +354,5 @@
 	<origin rpy="0 0 0" xyz="0 0 -0.5"/>
 </joint>
+ End of refactored things in the new .urdf.xacro (ABOVE IS DEPRECATED)-->
 <!-- !!!!!!!!!!!!!!!!!!!!!~~~~~~~Left Arm~~~~~~!!!!!!!!!!!!!!!!!!!!!!!!!!! -->
 <!-- Authors: Devon Ash, Jordan Balanko -->

Commit message: Added: integration of talos_common (unparsed and untested urdf)

File: talos_navigation/talos_description/urdf/talos_common.xacro (robot description, xacro)
@@ -1,508 +1,39 @@
 <?xml version="1.0"?>
-<robot xmlns:xacro="http://www.ros.org/wiki/xacro" name="talos">
-  <!-- Base Plate and Spokes -->
-<!-- Refactored already to the new .urdf.xacro, this code until ending specified is DEPRECATED
-  <link name="horizontal_base_plate">
-  	<visual>
-		<geometry>
-			<box size="0.40 0.20 0.03"/>
-		</geometry>
-		<origin rpy="0 0 1.57" xyz="0 0 0"/>
-		<material name="white">
-			<color rgba="1 1 1 1"/>
-		</material>
-	</visual>
-  </link>
-  <joint name="base_plate_to_base_bar" type="fixed">
-  	<parent link="horizontal_base_plate"/>
-	<child link="horizontal_base_plate_bar"/>
-	<origin xyz="0.1 0 0" rpy="0 0 0"/>
-  </joint>
-  <link name="horizontal_base_plate_bar">
-    <visual>
-	<geometry>
-		<box size="0.03 0.61905 0.03"/>
-	</geometry>
-	<origin rpy="0 0 0" xyz="0 0 0"/>
-	<material name="white">
-		<color rgba="1 1 1 1"/>
-	</material>
-    </visual>
-  </link>
-  <link name="lwheel_spoke">
-	<visual>
-		<geometry>
-			<cylinder length="0.07" radius="0.015"/>
-		</geometry>
-		<origin rpy="0 0 0" xyz="0 0 0"/>
-		<material name="white">
-			<color rgba="1 1 1 1"/>
-		</material>
-	</visual>
-  </link>
-  <link name="rwheel_spoke">
-	<visual>
-		<geometry>
-			<cylinder length="0.07" radius="0.015"/>
-		</geometry>
-		<origin rpy="0 0 0" xyz="0 0 0"/>
-		<material name="white">
-			<color rgba="1 1 1 1"/>
-		</material>
-	</visual>
-  </link>
-  <joint name="base_plate_to_lwheel_spoke" type="fixed">
-	<parent link="horizontal_base_plate"/>
-	<child link="lwheel_spoke"/>
-	<origin rpy="1.57 0 0" xyz="0 -0.235 0"/>
-  </joint>
-<joint name="base_plate_to_rwheel_spoke" type="fixed">
-	<parent link="horizontal_base_plate"/>
-	<child link="rwheel_spoke"/>
-	<origin rpy="1.57 0 0" xyz="0 0.235 0"/>
-</joint>
-  <link name="lwheel">
-	<visual>
-		<geometry>
-			<cylinder length="0.01" radius="0.0761"/>
-		</geometry>
-		<origin rpy="0 0 0" xyz="0 0 0"/>
-		<material name="black">
-			<color rgba="0 0 0 1"/>
-		</material>
-	</visual>
-  </link>
-  <link name="rwheel">
-	<visual>
-		<geometry>
-			<cylinder length="0.01" radius="0.0761"/>
-		</geometry>
-		<origin rpy="0 0 0" xyz="0 0 0"/>
-		<material name="black">
-			<color rgba="0 0 0 1"/>
-		</material>
-	</visual>
-  </link>
-  <joint name="lwheel_spoke_to_lwheel" type="fixed">
-	<parent link="lwheel_spoke"/>
-	<child link="lwheel"/>
-	<origin rpy="0 0 0" xyz="0 0 0.04"/>
-  </joint>
-  <joint name="rwheel_spoke_to_rwheel" type="fixed">
-	<parent link="rwheel_spoke"/>
-	<child link="rwheel"/>
-	<origin rpy="0 0 0" xyz="0 0 -0.04"/>
-  </joint>
-  <link name="lwheel_bottom_bar">
-	<visual>
-	<geometry>
-		<box size="0.03 0.61905 0.03"/>
-	</geometry>
-	<origin rpy="0 0 0" xyz="0 0 0"/>
-	<material name="white">
-		<color rgba="1 1 1 1"/>
-	</material>
-    </visual>
-  </link>
- <link name="rwheel_bottom_bar">
-	<visual>
-	<geometry>
-		<box size="0.03 0.61905 0.03"/>
-	</geometry>
-	<origin rpy="0 0 0" xyz="0 0 0"/>
-	<material name="white">
-		<color rgba="1 1 1 1"/>
-	</material>
-    </visual>
-  </link>
- <joint name="base_plate_bar_to_lwheel_bottom_bar" type="fixed">
-	<parent link="horizontal_base_plate_bar"/>
-	<child link="lwheel_bottom_bar"/>
-	<origin rpy="0 0 1.57" xyz="-0.295 -0.31 0"/>
-  </joint>
- <joint name="base_plate_bar_to_rwheel_bottom_bar" type="fixed">
-	<parent link="horizontal_base_plate_bar"/>
-	<child link="rwheel_bottom_bar"/>
-	<origin rpy="0 0 1.57" xyz="-0.295 0.31 0"/>
-  </joint>
-  <link name="bottom_bar_opposite_from_wheels">
-	<visual>
-	<geometry>
-		<box size="0.03 0.61905 0.03"/>
-	</geometry>
-	<origin rpy="0 0 0" xyz="0 0 0"/>
-	<material name="white">
-		<color rgba="0 0 0 1"/>
-	</material>
-    </visual>
-  </link>
-  <joint name="rwheel_bottom_bar_to_opposite_bottom_bar" type="fixed">
-	<parent link="rwheel_bottom_bar"/>
-	<child link="bottom_bar_opposite_from_wheels"/>
-	<origin rpy="0 0 1.57" xyz="-0.295 0.295 0"/>
-  </joint>
-  <joint name="lwheel_bottom_bar_to_opposite_bottom_bar" type="fixed">
-  	<parent link="lwheel_bottom_bar"/>
-	<child link="bottom_bar_opposite_from_wheels"/>
-	<origin rpy="0 0 0" xyz="0 0 0"/>
-  </joint>
-  <link name="opposite_vertical_rwheel_bar">
-	<visual>
-	<geometry>
-		<box size="0.03 0.32876 0.03"/>
-	</geometry>
-	<origin rpy="0 0 0" xyz="0 0 0"/>
-	<material name="white">
-		<color rgba="1 1 1 1"/>
-	</material>
-    </visual>
-  </link>
-  <joint name="rwheel_bottom_bar_to_ov_rwheel_bar" type="fixed">
-  	<parent link="rwheel_bottom_bar"/>
-	<child link="opposite_vertical_rwheel_bar"/>
-	<origin rpy="1.57 0 0" xyz="0 0.295 0.16438"/>
-  </joint>
-  <link name="opposite_vertical_lwheel_bar">
-	<visual>
-	<geometry>
-		<box size="0.03 0.32876 0.03"/>
-	</geometry>
-	<origin rpy="0 0 0" xyz="0 0 0"/>
-	<material name="white">
-		<color rgba="1 1 1 1"/>
-	</material>
-    </visual>
-  </link>
-<joint name="lwheel_bottom_bar_to_ov_lwheel_bar" type="fixed">
-  	<parent link="lwheel_bottom_bar"/>
-	<child link="opposite_vertical_lwheel_bar"/>
-	<origin rpy="1.57 0 0" xyz="0 0.295 0.16438"/>
-  </joint>
-<link name="vertical_lwheel_bar">
-	<visual>
-	<geometry>
-		<box size="0.03 0.32876 0.03"/>
-	</geometry>
-	<origin rpy="0 0 0" xyz="0 0 0"/>
-	<material name="white">
-		<color rgba="1 1 1 1"/>
-	</material>
-    </visual>
-  </link>
-<joint name="lwheel_bottom_bar_to_v_lwheel_bar" type="fixed">
-  	<parent link="lwheel_bottom_bar"/>
-	<child link="vertical_lwheel_bar"/>
-	<origin rpy="1.57 0 0" xyz="0 -0.295 0.16438"/>
-  </joint>
-<link name="vertical_rwheel_bar">
-	<visual>
-	<geometry>
-		<box size="0.03 0.32876 0.03"/>
-	</geometry>
-	<origin rpy="0 0 0" xyz="0 0 0"/>
-	<material name="white">
-		<color rgba="1 1 1 1"/>
-	</material>
-    </visual>
-  </link>
-<joint name="lwheel_bottom_bar_to_v_rwheel_bar" type="fixed">
-  	<parent link="rwheel_bottom_bar"/>
-	<child link="vertical_rwheel_bar"/>
-	<origin rpy="1.57 0 0" xyz="0 -0.295 0.16438"/>
-  </joint>
-<link name="top_plate">
-	<visual>
-	<geometry>
-		<box size="0.64905 0.61905 0.03"/>
-	</geometry>
-	<origin rpy="0 0 0" xyz="0 0 0"/>
-	<material name="white">
-		<color rgba="1 1 1 1"/>
-	</material>
-    </visual>
-  </link>
-<joint name="v_rwheel_bar_to_top_plate" type="fixed">
-  	<parent link="vertical_rwheel_bar"/>
-	<child link="top_plate"/>
-	<origin rpy="1.57 0 0" xyz="-0.31 0.16438 -0.294525"/>
-  </joint>
-<joint name="v_lwheel_bar_to_top_plate" type="fixed">
-  	<parent link="vertical_lwheel_bar"/>
-	<child link="top_plate"/>
-	<origin rpy="0 0 0" xyz="0 0 0"/>
-  </joint>
-<joint name="opposite__vertical_lwheel_bar_to_top_plate" type="fixed">
-  	<parent link="opposite_vertical_lwheel_bar"/>
-	<child link="top_plate"/>
-	<origin rpy="0 0 0" xyz="0 0 0"/>
-  </joint>
-<joint name="opposite__vertical_rwheel_bar_to_top_plate" type="fixed">
-  	<parent link="opposite_vertical_rwheel_bar"/>
-	<child link="top_plate"/>
-	<origin rpy="0 0 0" xyz="0 0 0"/>
-  </joint>
-<link name="right_castor_spoke">
-	<visual>
-		<geometry>
-			<cylinder length="0.07" radius="0.015"/>
-		</geometry>
-		<origin rpy="0 0 0" xyz="0 0 0"/>
-		<material name="white">
-			<color rgba="1 1 1 1"/>
-		</material>
-	</visual>
-  </link>
-<link name="left_castor_spoke">
-	<visual>
-		<geometry>
-			<cylinder length="0.07" radius="0.015"/>
-		</geometry>
-		<origin rpy="0 0 0" xyz="0 0 0"/>
-		<material name="white">
-			<color rgba="1 1 1 1"/>
-		</material>
-	</visual>
-  </link>
-<joint name="rwheel_bottom_bar_to_rwheel_castor_spoke" type="fixed">
-  	<parent link="rwheel_bottom_bar"/>
-	<child link="right_castor_spoke"/>
-	<origin rpy="0 1.57 0" xyz="-0.035 0.2 0"/>
-  </joint>
-<joint name="lwheel_bottom_bar_to_lwheel_castor_spoke" type="fixed">
-  	<parent link="lwheel_bottom_bar"/>
-	<child link="left_castor_spoke"/>
-	<origin rpy="0 1.57 0" xyz="0.035 0.2 0"/>
-  </joint>
-<link name="right_castor_wheel">
-	<visual>
-		<geometry>
-			<cylinder length="0.01" radius="0.0761"/>
-		</geometry>
-		<origin rpy="0 0 0" xyz="0 0 0"/>
-		<material name="black">
-			<color rgba="0 0 0 1"/>
-		</material>
-	</visual>
-  </link>
-<link name="left_castor_wheel">
-	<visual>
-		<geometry>
-			<cylinder length="0.01" radius="0.0761"/>
-		</geometry>
-		<origin rpy="0 0 0" xyz="0 0 0"/>
-		<material name="black">
-			<color rgba="0 0 0 1"/>
-		</material>
-	</visual>
-  </link>
-<joint name="right_castor_spoke_to_right_castor_wheel" type="fixed">
-  	<parent link="right_castor_spoke"/>
-	<child link="right_castor_wheel"/>
-	<origin rpy="0 0 0" xyz="0 0 -0.03805"/>
-  </joint>
-<joint name="left_castor_spoke_to_left_castor_wheel" type="fixed">
-  	<parent link="left_castor_spoke"/>
-	<child link="left_castor_wheel"/>
-	<origin rpy="0 0 0" xyz="0 0 0.03805"/>
-  </joint>
-<link name="rotational_base_plate">
-	<visual>
-		<geometry>
-			<cylinder length="0.01" radius="0.15"/>
-		</geometry>
-		<origin rpy="0 0 0" xyz="0 0 0"/>
-		<material name="black">
-			<color rgba="0 0 0 1"/>
-		</material>
-	</visual>
-  </link>
-<joint name="top_plate_to_rotational_base" type="fixed">
-  	<parent link="top_plate"/>
-	<child link="rotational_base_plate"/>
-	<origin rpy="0 0 0" xyz="0 0 -0.015"/>
-</joint>
-<link name="top_rotating_plate">
-	<visual>
-		<geometry>
-			<cylinder length="0.01" radius="0.15"/>
-		</geometry>
-		<origin rpy="0 0 0" xyz="0 0 0"/>
-		<material name="black">
-			<color rgba="1 0 0 -0.015"/>
-		</material>
-	</visual>
-  </link>
-<joint name="rotational_base_connection" type="fixed">
-  	<parent link="rotational_base_plate"/>
-	<child link="top_rotating_plate"/>
-	<origin rpy="0 0 0" xyz="0 0 0"/>
-</joint>
-  <link name="body">
-	<visual>
-	<geometry>
-		<box size="0.4 0.4 1.0"/>
-	</geometry>
-	<origin rpy="0 0 0" xyz="0 0 0"/>
-	<material name="white">
-		<color rgba="1 1 1 1"/>
-	</material>
-    </visual>
-  </link>
-<joint name="top_rotating_plate_to_body" type="fixed">
-  	<parent link="top_rotating_plate"/>
-	<child link="body"/>
-	<origin rpy="0 0 0" xyz="0 0 -0.5"/>
-</joint>
- End of refactored things in the new .urdf.xacro (ABOVE IS DEPRECATED)-->
-<!-- !!!!!!!!!!!!!!!!!!!!!~~~~~~~Left Arm~~~~~~!!!!!!!!!!!!!!!!!!!!!!!!!!! -->
-<!-- Authors: Devon Ash, Jordan Balanko -->
+<!-- Author: Devon Ash -->
 <!-- Maintainer: noobaca2@gmail.com -->
- <link name="left_shoulder">
-	<!-- TODO: Jordan start -->
-	<!-- TODO Jordan: Please fill in the required values specified by "0" or near approximations -->
-	<inertial>
-		<mass value="0" />
-		<origin xyz="0 0 0" />
-		<inertia ixx="0" ixy="0" ixz="0"
-			  iyy="0" iyz="0"
-			  izz="0" />
-	</inertial>
-        <!-- TODO: Jordan end -->
-        <!-- TODO: Someone? Not sure how these are done yet. -->
-	<collision>
-		<origin xyz="0 0 0" rpy="0 0 0" />
-		<geometry>
-		  <!-- <mesh filename="package://pr2_description/meshes/upper_arm_v0/elbow_flex.stl" /> -->
-		</geometry>
-	</collision>
-	<visual>
-		<geometry>
-			<box size="0.2 0.1 0.22"/>
-		</geometry>
-		<origin rpy="0 0 0" xyz="0 0 0"/>
-		<!-- TODO: Add meshes -->
-		<material name="white">
-			<color rgba="1 1 1 1"/>
-		</material>
-	</visual>
-</link>
-<joint name="body_to_left_shoulder" type="fixed">
-	<!-- Note: Crude approximation of physical robot -->
-  	<parent link="body"/>
-	<child link="left_shoulder"/>
-	<origin rpy="0 0 1.57" xyz="-0.25 -0.1 -0.39"/>
- 	<!-- TODO Jordan Start: -->
-        <!-- TODO Jordan: Please fill in the required values specified by "?" or near approximations -->
-	<!-- Note: Code template taken from PR2_upper_arm.urdf for templating -->
-	<!-- Doc: axis of revolution -->
-	<axis xyz="0 1 0" />
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