Commit message: Added: Talos tilting base laser

File: talos_navigation/talos_description/urdf/talos_common.urdf.xacro (robot description, xacro)
@@ -18,4 +18,5 @@
 <xacro:include filename="$(find talos_navigation)/talos_description/urdf/base_v0/talos_base.urdf.xacro" />
 <xacro:include filename="$(find talos_navigation)/talos_description/urdf/head_v0/talos_head.urdf.xacro" />
+<xacro:include filename="$(find talos_navigation)/talos_description/urdf/tilting_laser_v0/talos_tilting_laser.urdf.xacro" />
 <!-- Use the macros defined in the xacro above to define actual urdf -->
 <!--                                               -->
@@ -31,4 +32,7 @@
 <property name="talos_head_offset_y" value="0" />
 <property name="talos_head_offset_z" value="0" />
+<property name="talos_base_laser_x" value="0" />
+<property name="talos_base_laser_y" value="0.15" />
+<property name="talos_base_laser_z" value="0.3" />
 <!--                                               -->
 <!--                 TALOS  DEFINITION             -->
@@ -46,3 +50,7 @@
 	<origin xyz="${talos_head_offset_x} ${talos_head_offset_y} ${talos_head_offset_z}" rpy="0 0 0" />
 </xacro:talos_head>
+<!-- Instantiates the base laser -->
+<xacro:talos_tilting_laser>
+	<origin xyz="${talos_base_laser_x} ${talos_base_laser_y} ${talos_base_laser_z}" rpy="0 0 0" />
+</xacro:talos_tilting_laser>
 </robot>

Commit message: Fixed: Bug to do with spawning laser and bugged xacro:include line

File: talos_navigation/talos_description/urdf/talos_common.urdf.xacro (robot description, xacro)
@@ -32,7 +32,4 @@
 <property name="talos_head_offset_y" value="0" />
 <property name="talos_head_offset_z" value="0" />
-<property name="talos_base_laser_x" value="0" />
-<property name="talos_base_laser_y" value="0.15" />
-<property name="talos_base_laser_z" value="0.3" />
 <!--                                               -->
 <!--                 TALOS  DEFINITION             -->
@@ -51,6 +48,3 @@
 </xacro:talos_head>
 <!-- Instantiates the base laser -->
-<xacro:talos_tilting_laser>
-	<origin xyz="${talos_base_laser_x} ${talos_base_laser_y} ${talos_base_laser_z}" rpy="0 0 0" />
-</xacro:talos_tilting_laser>
 </robot>

File: talos_navigation/talos_description/urdf/tilting_laser_v0/talos_tilting_laser.urdf.xacro (robot description, xacro)
@@ -11,15 +11,38 @@
 <!--               GENERAL CONSTANTS               -->
 <!--                                               -->
+<property name="talos_base_laser_x" value="0" />
+<property name="talos_base_laser_y" value="0.15" />
+<property name="talos_base_laser_z" value="0.3" />
 <property name="M_PI" value="3.1415926535897931"/>
-<xacro:macro name="talos_base_laser" params="*origin">
   <!-- base laser -->
-    <xacro:hokuyo_lx30_laser_v0 name="talos_base_laser_link" parent="talos_base" ros_topic="base_scan" update_rate="20" min_angle="-2.2689" max_angle="2.2689" >
-      <xacro:insert_block name="origin" />
+    <xacro:hokuyo_lx30_laser_v0 name="talos_base_laser" parent="talos_base" ros_topic="base_scan" update_rate="20" min_angle="-2.2689" max_angle="2.2689" >
+      <origin xyz="${talos_base_laser_x} ${talos_base_laser_y} ${talos_base_laser_z}" rpy="0 0 0" />
     </xacro:hokuyo_lx30_laser_v0>
 <joint name="talos_base_laser_joint" type="fixed">
     <origin xyz="0 0 0" rpy="0 0 0" />
-    <parent link="talos_base" />
-    <child link="talos_base_laser_link"/>
+    <parent link="talos_base_laser_link" />
+    <child link="talos_base_laser_simulator_link"/>
   </joint>
-</xacro:macro>
+<!-- This allows us to see it in rviz/gazebo -->
+<link name="talos_base_laser_simulator_link">
+    <inertial>
+      <mass value="0.01" />
+      <origin xyz="0 0 0" />
+      <inertia ixx="0.001"  ixy="0.0"  ixz="0.0"
+               iyy="0.001"  iyz="0.0"
+               izz="0.001" />
+    </inertial>
+    <visual>
+      <origin xyz="0 0 0" rpy="0 0 0"/>
+      <geometry>
+        <box size="0.05 0.05 0.1" />
+      </geometry>
+    </visual>
+    <collision>
+      <origin xyz="0 0 0" rpy="0 0 0"/>
+      <geometry>
+        <box size="0.05 0.05 0.1" />
+      </geometry>
+    </collision>
+  </link>
 </robot>
