Commit message: Added: fixed bugs inside of the committed files regarding parsing of urdf

File: talos_navigation/talos_description/urdf/talos_common.urdf (robot description, URDF)
Before this commit: robot talos, 9 links, 8 joints
Links:
- link left_upper_arm_link: geometry visual box size=0.47 0.2 0.22

File: talos_navigation/talos_description/urdf/talos_common.urdf.xacro (robot description, xacro)
@@ -14,7 +14,7 @@
 <!--                 INCLUDED XACROS               -->
 <!--                                               -->
-<xacro:include filename="$(find talos_navigation)/talos_description/urdf/talos_torso.urdf.xacro" />
-<xacro:include filename="$(find talos_navigation)/talos_description/urdf/talos_upper_arm_v1.urdf.xacro" />
-<xacro:include filename="$(find_talos_navigation)/talos_description/urdf/talos_base.urdf.xacro" />
+<xacro:include filename="$(find talos_navigation)/talos_description/urdf/torso_v0/talos_torso.urdf.xacro" />
+<xacro:include filename="$(find talos_navigation)/talos_description/urdf/upper_arm_v0/talos_upper_arm_v1.urdf.xacro" />
+<xacro:include filename="$(find talos_navigation)/talos_description/urdf/base_v0/talos_base.urdf.xacro" />
 <!-- Use the macros defined in the xacro above to define actual urdf -->
 <!--                                               -->

File: talos_navigation/talos_description/urdf/upper_arm_v0/talos_upper_arm_v1.urdf.xacro (robot description, xacro)
@@ -110,5 +110,5 @@
 	<visual>
 		<geometry>
-			<box size="${upper_arm_length}=.47 ${upper_arm_width}=0.2 ${upper_arm_height}0.22"/>
+			<box size="${upper_arm_length} ${upper_arm_width} ${upper_arm_height}"/>
 		</geometry>
 		<origin rpy="0 0 0" xyz="0 0 0"/>

Commit message: Modified: fixed bug regarding tf tree

File: talos_navigation/talos_description/urdf/talos_common.urdf (robot description, URDF)
Before this commit: robot talos, 9 links, 8 joints
Links:
- added link head_pan_link; visual box size=0 0 0
- added link head_tilt_link; visual box size=0.1 0.1 0.1
Joints:
- added joint head_pan_joint: type continuous, parent torso_link, child head_pan_link, origin xyz=0 0 0 rpy=0 0 0, axis 0 0 1, limit effort=10 velocity=10
- added joint head_tilt_joint: type revolute, parent head_pan_link, child head_tilt_link, origin xyz=0 0 0 rpy=0 0 0, axis 0 1 0, limit lower=-1 upper=1 effort=10 velocity=10

File: talos_navigation/talos_description/urdf/talos_common.urdf.xacro (robot description, xacro)
@@ -43,5 +43,5 @@
 <xacro:talos_upper_arm side="left" parent="torso_link" reflect="1" />
 <!-- Instantiates talos head -->
-<xacro:talos_head parent="talos_torso_link">
+<xacro:talos_head parent="torso_link">
 	<origin xyz="${talos_head_offset_x} ${talos_head_offset_y} ${talos_head_offset_z}" rpy="0 0 0" />
 </xacro:talos_head>

Commit message: Modified: Talos_common had an errror Bug fix: Fixed by hacking a joint and a link into talos laser .urdf.xacro

File: talos_navigation/talos_description/urdf/talos_common.urdf (robot description, URDF)
Before this commit: robot talos, 11 links, 10 joints
Links:
- added link talos_base_laser_link, mass 0.001
- added link talos_base_laser_simulator_link, mass 0.01; collision box size=0.05 0.05 0.1; visual box size=0.05 0.05 0.1
- added link talos_base_link; visual box size=0 0 0
Joints:
- added joint talos_base_laser_joint: type fixed, parent talos_base_link, child talos_base_laser_link, origin xyz=0 0.15 0.3 rpy=0 0 0, axis 0 1 0
- added joint talos_base_laser_simulator_joint: type fixed, parent talos_base_laser_link, child talos_base_laser_simulator_link, origin xyz=0 0 0 rpy=0 0 0
- added joint talos_base_link_hack: type fixed, parent talos_base, child talos_base_link, origin xyz=0 0 0 rpy=0 0 0

File: talos_navigation/talos_description/urdf/tilting_laser_v0/talos_tilting_laser.urdf.xacro (robot description, xacro)
@@ -15,9 +15,24 @@
 <property name="talos_base_laser_z" value="0.3" />
 <property name="M_PI" value="3.1415926535897931"/>
-  <!-- base laser -->
+<!-- Small hack to get around the fact that hokuyo xacro adds a _link to the parent name -->
+<link name="talos_base_link">
+    <visual>
+      <origin xyz="0 0 0" rpy="0 0 0"/>
+      <geometry>
+        <box size="0 0 0" />
+      </geometry>
+    </visual>
+</link>
+<joint name="talos_base_link_hack" type="fixed">
+ <origin xyz="0 0 0" rpy="0 0 0" />
+    <parent link="talos_base" />
+    <child link="talos_base_link"/>
+</joint>
+<!-- End of hack -->
+<!-- base laser -->
     <xacro:hokuyo_lx30_laser_v0 name="talos_base_laser" parent="talos_base" ros_topic="base_scan" update_rate="20" min_angle="-2.2689" max_angle="2.2689" >
       <origin xyz="${talos_base_laser_x} ${talos_base_laser_y} ${talos_base_laser_z}" rpy="0 0 0" />
     </xacro:hokuyo_lx30_laser_v0>
-<joint name="talos_base_laser_joint" type="fixed">
+<joint name="talos_base_laser_simulator_joint" type="fixed">
     <origin xyz="0 0 0" rpy="0 0 0" />
     <parent link="talos_base_laser_link" />

Commit message: Added: base laser now in correct coordinate frame

File: talos_navigation/talos_description/urdf/talos_common.urdf (robot description, URDF)
Before this commit: robot talos, 13 links, 12 joints
Joints:
- joint talos_base_laser_joint: origin xyz=0 0.15 0.3 rpy=0 0 0 -> xyz=0 0.15 0 rpy=0 0 0

File: talos_navigation/talos_description/urdf/tilting_laser_v0/talos_tilting_laser.urdf.xacro (robot description, xacro)
@@ -13,5 +13,5 @@
 <property name="talos_base_laser_x" value="0" />
 <property name="talos_base_laser_y" value="0.15" />
-<property name="talos_base_laser_z" value="0.3" />
+<property name="talos_base_laser_z" value="0" />
 <property name="M_PI" value="3.1415926535897931"/>
 <!-- No longer need small hack, DEPRECATED
