Commit message: Added: modifications to parse

File: talos_navigation/talos_description/urdf/head_v0/talos_head.urdf.xacro (robot description, xacro)
@@ -125,7 +125,7 @@
 <!--                                               -->
 <!-- Instantiate the head of talos -->
-<xacro:macro name="talos_head" params="name parent *origin">
+<xacro:macro name="talos_head" params="parent *origin">
 	<!-- Instantiate the head_pan of talos -->
-	<xacro:talos_head_pan name="${name}" parent="${parent}">
+	<xacro:talos_head_pan name="head_pan" parent="${parent}">
 		<insert_block name="origin" />
 	</xacro:talos_head>

File: talos_navigation/talos_description/urdf/talos_common.urdf.xacro (robot description, xacro)
@@ -17,4 +17,5 @@
 <xacro:include filename="$(find talos_navigation)/talos_description/urdf/upper_arm_v0/talos_upper_arm_v1.urdf.xacro" />
 <xacro:include filename="$(find talos_navigation)/talos_description/urdf/base_v0/talos_base.urdf.xacro" />
+<xacro:include fliename="$(find talos_navigation)/talos_description/urdf/head_v0/talos_head.urdf.xacro" />
 <!-- Use the macros defined in the xacro above to define actual urdf -->
 <!--                                               -->
@@ -26,4 +27,8 @@
 <!-- VALUE: Torso height/2 + base height -->
 <property name="torso_offset_z" value="0.5" />
+<!-- TODO: Measure proper offsets for taloshead -->
+<property name="talos_head_offset_x" value="0" />
+<property name="talos_head_offset_y" value="0" />
+<property name="talos_head_offset_z" value="0" />
 <!--                                               -->
 <!--                 TALOS  DEFINITION             -->
@@ -37,3 +42,7 @@
 <!-- Instantiates the upper arm of talos -->
 <xacro:talos_upper_arm side="left" parent="torso_link" reflect="1" />
+<!-- Instantiates talos head -->
+<xacro:talos_head parent="talos_torso_link">
+	<origin xyz="${talos_head_offset_x} ${talos_head_offset_y} ${talos_head_offset_z}" rpy="0 0 0" />
+</xacro:talos_head>
 </robot>

Commit message: Fixed: Bug in talos_head giving parsing errors Fixed: overall talos_common bug, include erro

File: talos_navigation/talos_description/urdf/head_v0/talos_head.urdf.xacro (robot description, xacro)
@@ -6,5 +6,5 @@
        xmlns:controller="http://playerstage.sourceforge.net/gazebo/xmlschema/#controller"
        xmlns:interface="http://playerstage.sourceforge.net/gazebo/xmlschema/#interface"
-       xmlns:xacro="http://ros.org/wiki/xacro">
+       xmlns:xacro="http://ros.org/wiki/xacro" name="talos_head">
 <!--                                               -->
 <!--               GENERAL CONSTANTS               -->
@@ -32,22 +32,24 @@
 <!--                                               -->
 <xacro:macro name="talos_head_pan" params="name parent *origin">
-<joint name="${name}_joint" type="continuous" />
+<joint name="${name}_joint" type="continuous">
 	<parent link="${parent}"/>
 	<child link="${name}_link"/>
-	<xacro:insert block_name="origin"/>
+	<xacro:insert_block name="origin"/>
 	<axis xyz="0 0 1" />
-       <limit effort="${max_head_pan_effort}" velocity="${max_head_pan_velocity}"/> <!-- alpha tested effort and velocity limits -->
-       <safety_controller k_velocity="${head_pan_safety_k_velocity}" />
-       <dynamics damping="${head_pan_damping}" friction="${head_pan_friction}" />
+       <limit effort="${max_head_pan_effort}" velocity="${max_head_pan_velocity}" />
+	<!-- TODO: Not sure what this is -->
+      <!--  <safety_controller k_velocity="${head_pan_safety_k_velocity}" /> -->
+	<!-- TODO: set proper values first -->
+       <!-- <dynamics damping="${head_pan_damping}" friction="${head_pan_friction}" /> -->
 </joint>
 <link name="${name}_link">
 	<!-- TODO: Fill in constants above related to inertia -->
-      <inertial>
+      <!-- <inertial>
         <mass value="${head_pan_link_mass}" />
         <origin xyz="0 0 0" rpy="0 0 0" />
- 	<!-- These are the incorrect inertias -->
+ 	TODO: These are the incorrect inertias
         <inertia ixx="0.032497592" ixy="0.00063604088" ixz="0.0025851534"
                  iyy="0.046545627" iyz="-0.0024534295" izz="0.057652724" />
-      </inertial>
+      </inertial> -->
       <visual>
         <origin xyz="0 0 0.0" rpy="0 0 0 " />
@@ -58,4 +60,5 @@
 	<!-- TODO: Approximation -->
         <geometry>
+		<box size="0 0 0" />
 	</geometry>
         <material name="Blue" />
@@ -67,5 +70,5 @@
         </geometry>
       </collision> -->
-    </link>
+</link>
 <!-- extensions -->
 <!-- TODO: Add transmissions here
@@ -128,11 +131,11 @@
 	<!-- Instantiate the head_pan of talos -->
 	<xacro:talos_head_pan name="head_pan" parent="${parent}">
-		<insert_block name="origin" />
-	</xacro:talos_head>
+		<xacro:insert_block name="origin" />
+	</xacro:talos_head_pan>
 	<!-- Instantiate the head tilt of talos -->
 	<xacro:talos_head_tilt name="head_tilt" parent="head_pan_link">
 		<!-- TODO: Proper positioning of tilt mechanism -->
 		<origin xyz="0 0 0" rpy="0 0 0" />
-	</xacro:talos_head>
+	</xacro:talos_head_tilt>
 </xacro:macro>
 </robot>

File: talos_navigation/talos_description/urdf/talos_common.urdf.xacro (robot description, xacro)
@@ -17,5 +17,5 @@
 <xacro:include filename="$(find talos_navigation)/talos_description/urdf/upper_arm_v0/talos_upper_arm_v1.urdf.xacro" />
 <xacro:include filename="$(find talos_navigation)/talos_description/urdf/base_v0/talos_base.urdf.xacro" />
-<xacro:include fliename="$(find talos_navigation)/talos_description/urdf/head_v0/talos_head.urdf.xacro" />
+<xacro:include filename="$(find talos_navigation)/talos_description/urdf/head_v0/talos_head.urdf.xacro" />
 <!-- Use the macros defined in the xacro above to define actual urdf -->
 <!--                                               -->
