Commit message: Modified: things

File: talos_navigation/talos_description/urdf/tilting_laser_v0/talos_tilting_laser.urdf.xacro (robot description, xacro)
@@ -17,4 +17,9 @@
       <xacro:insert_block name="origin" />
     </xacro:hokuyo_lx30_laser_v0>
+<joint name="talos_base_laser_joint" type="fixed">
+    <origin xyz="0 0 0" rpy="0 0 0" />
+    <parent link="talos_base" />
+    <child link="talos_base_laser_link"/>
+  </joint>
 </xacro:macro>
 </robot>

Commit message: Things

File: talos_navigation/talos_description/urdf/tilting_laser_v0/talos_tilting_laser.urdf.xacro (robot description, xacro)
@@ -15,5 +15,5 @@
 <property name="talos_base_laser_z" value="0.3" />
 <property name="M_PI" value="3.1415926535897931"/>
-<!-- Small hack to get around the fact that hokuyo xacro adds a _link to the parent name -->
+Small hack to get around the fact that hokuyo xacro adds a _link to the parent name
 <link name="talos_base_link">
     <visual>
@@ -24,9 +24,10 @@
     </visual>
 </link>
+<!--
 <joint name="talos_base_link_hack" type="fixed">
  <origin xyz="0 0 0" rpy="0 0 0" />
     <parent link="talos_base" />
     <child link="talos_base_link"/>
-</joint>
+</joint> -->
 <!-- End of hack -->
 <!-- base laser -->
