Commit message: Added: Completed talos_base.urdf except for the TODO's in the file. Will make issue for these

File: talos_navigation/talos_description/urdf/base_v0/talos_base.urdf.xacro (robot description, xacro)
@@ -2,4 +2,5 @@
 <!-- Author: Devon Ash -->
 <!-- Maintainer: noobaca2@gmail.com -->
+<!-- TODO: Smoke Test this file in gazebo and RVIZ! -->
 <robot xmlns:sensor="http://playerstage.sourceforge.net/gazebo/xmlschema/#sensor"
        xmlns:controller="http://playerstage.sourceforge.net/gazebo/xmlschema/#controller"
@@ -18,11 +19,11 @@
   <property name="caster_offset_z" value="0.0282" />
 -->
-<!--               General constants               -->
-<!--               General constants               -->
-<!--               General constants               -->
+<!--                                               -->
+<!--               GENERAL CONSTANTS               -->
+<!--                                               -->
 <property name="M_PI" value="3.1415926535897931"/>
-<!--               Wheel constants                 -->
-<!--               Wheel constants                 -->
-<!--               Wheel constants                 -->
+<!--                                               -->
+<!--               WHEEL CONSTANTS                 -->
+<!--                                               -->
 <property name="wheel_thickness" value="0.01"/>
 <property name="wheel_radius" value="0.0761"/>
@@ -32,7 +33,19 @@
 <property name="max_wheel_effort" value="7" />
 <property name="max_wheel_velocity" value="15" />
-<!--                     Wheel definition (For all 4)             -->
-<!--                     Wheel definition (For all 4)             -->
-<!--                     Wheel definition (For all 4)             -->
+<!--                                               -->
+<!--                 BASE CONSTANTS                -->
+<!--                                               -->
+<!-- TODO: Accurate and precise values or approximations to be filled in -->
+<property name="talos_base_mass" value="0" />
+<property name="talos_base_cg_x" value="0" />
+<property name="talos_base_cg_y" value="0" />
+<property name="talos_base_cg_z" value="0" />
+<property name="talos_base_collision_size_z" value="0" />
+<property name="talos_base_lazer_x" value="0" />
+<property name="talos_base_lazer_y" value="0" />
+<property name="talos_base_lazer_z" value="0" />
+<!--                                               -->
+<!--                WHEEL DEFINITION               -->
+<!--                                               -->
 <xacro:macro name="talos_wheel" params="suffix parent reflect">
 <joint name="${parent}_${suffix}_wheel_joint" type="continuous">
@@ -84,3 +97,72 @@
  -->
 </xacro:macro>
+<!--                       Base Definition                 -->
+<!--                       Base Definition                 -->
+<!--                       Base Definition                 -->
+<xacro:macro name="talos_base" params="name">
+<link name="${name}_base_plate">
+	<!-- TODO: Jordan to put proper values for the xml below
+	<inertial>
+        <mass value="${talos_base_mass}" />
+        <origin xyz="${talos_base_cg_x} ${talos_base_cg_y} ${talos_base_cg_z}" />
+        <inertia ixx="5.652232699207" ixy="-0.009719934438" ixz="1.293988226423"
+                 iyy="5.669473158652" iyz="-0.007379583694" izz="3.683196351726" />
+      </inertial>
+      -->
+  	<visual>
+              <!-- TODO: Replace with .dae file -->
+		<geometry>
+			<box size="${talos_base_width} ${talos_base_length} ${talos_base_height}"/>
+		</geometry>
+		<origin rpy="0 0 0" xyz="0 0 0"/>
+              <!-- TODO: Replace with .stl file -->
+		<material name="white">
+			<color rgba="1 1 1 1"/>
+		</material>
+	</visual>
+   <!-- TODO: Add collisions
+   <collision>
+        <origin xyz="0 0 0" rpy="0 0 0" />
+	 <!-- TODO: Replace with .stl file
+        <geometry>
+          <mesh filename="package://pr2_description/meshes/base_v0/base_L.stl" />
+        </geometry>
+      </collision>
+    -->
+</link>
+<!-- talos_base_footprint is a fictitious link(frame) that is on the ground right below base_link origin,
+navigation stack dedpends on this frame -->
+<link name="${name}_base_footprint">
+      <inertial>
+        <mass value="1.0" />
+        <origin xyz="0 0 0" />
+        <inertia ixx="0.01" ixy="0.0" ixz="0.0"
+                 iyy="0.01" iyz="0.0" izz="0.01" />
+      </inertial>
+      <visual>
+        <origin xyz="0 0 0" rpy="0 0 0" />
+        <geometry>
+          <box size="0.01 0.01 0.01" />
+        </geometry>
+        <material name="White" />
+      </visual>
+      <collision>
+        <!-- represent base collision with a simple rectangular model, positioned by base_size_z s.t. top
+surface of the collision box matches the top surface of the PR2 base -->
+        <origin xyz="0 0 ${0.051+base_collision_size_z/2}" rpy="0 0 0" />
+        <geometry>
+          <box size="0.001 0.001 0.001" />
+        </geometry>
+      </collision>
+    </link>
+    <joint name="${name}_base_footprint_joint" type="fixed">
+      <origin xyz="0 0 0.051" rpy="0 0 0" />
+      <child link="${name}_base_plate" />
+      <parent link="${name}_base_footprint"/>
+    </joint>
+  <!-- base laser -->
+    <xacro:hokuyo_lx30_laser_v0 name="${name}_base_laser" parent="${name}" ros_topic="base_scan" update_rate="20" min_angle="-2.2689" max_angle="2.2689" >
+      <origin xyz="${talos_base_laser_x} ${talos_base_laser_y} ${base_laser_z}" rpy="0 0 0" />
+    </xacro:hokuyo_lx30_laser_v0>
+</xacro:macro>
 </robot>

Commit message: Added: Talos wheels to the talos base

File: talos_navigation/talos_description/urdf/base_v0/talos_base.urdf.xacro (robot description, xacro)
@@ -101,5 +101,5 @@
 <!--                       Base Definition                 -->
 <xacro:macro name="talos_base" params="name">
-<link name="${name}_base_plate">
+<link name="talos_base">
 	<!-- TODO: Jordan to put proper values for the xml below
 	<inertial>
@@ -158,11 +158,16 @@
     <joint name="${name}_base_footprint_joint" type="fixed">
       <origin xyz="0 0 0.051" rpy="0 0 0" />
-      <child link="${name}_base_plate" />
+      <child link="talos_base" />
       <parent link="${name}_base_footprint"/>
     </joint>
   <!-- base laser -->
-    <xacro:hokuyo_lx30_laser_v0 name="${name}_base_laser" parent="${name}" ros_topic="base_scan" update_rate="20" min_angle="-2.2689" max_angle="2.2689" >
+    <xacro:hokuyo_lx30_laser_v0 name="${name}_base_laser" parent="talos_base" ros_topic="base_scan" update_rate="20" min_angle="-2.2689" max_angle="2.2689" >
       <origin xyz="${talos_base_laser_x} ${talos_base_laser_y} ${base_laser_z}" rpy="0 0 0" />
     </xacro:hokuyo_lx30_laser_v0>
+ <!-- Adding TALOS wheels to the base -->
+<xacro:talos_wheel suffix="fl" parent="talos_base" reflect="1" />
+<xacro:talos_wheel suffix="fr" parent="talos_base" reflect="-1" />
+<xacro:talos_wheel suffix="bl" parent="talos_base" reflect="1" />
+<xacro:talos_wheel suffix="br" parent="talos_base" reflect="-1" />
 </xacro:macro>
 </robot>

Commit message: Added: .urdf.xacro now compiles

File: talos_navigation/talos_description/urdf/base_v0/talos_base.urdf.xacro (robot description, xacro)
@@ -7,5 +7,5 @@
        xmlns:interface="http://playerstage.sourceforge.net/gazebo/xmlschema/#interface"
        xmlns:xacro="http://ros.org/wiki/xacro">
-<!-- Example includes
+<!-- Example includes  <
 <xacro:include filename="$(find pr2_description)/urdf/sensors/hokuyo_lx30_laser.urdf.xacro" />
 <xacro:include filename="$(find pr2_description)/urdf/base_v0/base.gazebo.xacro" />
@@ -42,7 +42,11 @@
 <property name="talos_base_cg_z" value="0" />
 <property name="talos_base_collision_size_z" value="0" />
-<property name="talos_base_lazer_x" value="0" />
-<property name="talos_base_lazer_y" value="0" />
-<property name="talos_base_lazer_z" value="0" />
+<!-- TODO: Input proper values here -->
+<property name="talos_base_width" value="0" />
+<property name="talos_base_height" value="0" />
+<property name="talos_base_length" value="0" />
+<property name="talos_base_laser_x" value="0" />
+<property name="talos_base_laser_y" value="0" />
+<property name="talos_base_laser_z" value="0" />
 <!--                                               -->
 <!--                WHEEL DEFINITION               -->
@@ -124,5 +128,5 @@
    <collision>
         <origin xyz="0 0 0" rpy="0 0 0" />
-	 <!-- TODO: Replace with .stl file
+	 TODO: Replace with .stl file
         <geometry>
           <mesh filename="package://pr2_description/meshes/base_v0/base_L.stl" />
@@ -150,5 +154,5 @@
         <!-- represent base collision with a simple rectangular model, positioned by base_size_z s.t. top
 surface of the collision box matches the top surface of the PR2 base -->
-        <origin xyz="0 0 ${0.051+base_collision_size_z/2}" rpy="0 0 0" />
+        <origin xyz="0 0 ${0.051+talos_base_collision_size_z/2}" rpy="0 0 0" />
         <geometry>
           <box size="0.001 0.001 0.001" />
@@ -163,5 +167,5 @@
   <!-- base laser -->
     <xacro:hokuyo_lx30_laser_v0 name="${name}_base_laser" parent="talos_base" ros_topic="base_scan" update_rate="20" min_angle="-2.2689" max_angle="2.2689" >
-      <origin xyz="${talos_base_laser_x} ${talos_base_laser_y} ${base_laser_z}" rpy="0 0 0" />
+      <origin xyz="${talos_base_laser_x} ${talos_base_laser_y} ${talos_base_laser_z}" rpy="0 0 0" />
     </xacro:hokuyo_lx30_laser_v0>
  <!-- Adding TALOS wheels to the base -->

File: talos_navigation/talos_description/urdf/upper_arm_v0/talos_upper_arm_v1.urdf.xacro (robot description, xacro)
@@ -6,5 +6,5 @@
        xmlns:controller="http://playerstage.sourceforge.net/gazebo/xmlschema/#controller"
        xmlns:interface="http://playerstage.sourceforge.net/gazebo/xmlschema/#interface"
-       xmlns:xacro="http://ros.org/wiki/xacro">
+       xmlns:xacro="http://ros.org/wiki/xacro" name="talos">
  <!-- Things that are needed only for Gazebo (not the physical robot). These include
 sensor and controller plugin specifications -->
@@ -121,2 +121,3 @@
 </link>
 </xacro:macro>
+</robot>

Commit message: Fixed: I promise, there are no parsing errors anymore! The values of the urdf haven't been properly set, however

File: talos_navigation/talos_description/urdf/base_v0/talos_base.urdf.xacro (robot description, xacro)
@@ -54,5 +54,5 @@
 <xacro:macro name="talos_wheel" params="suffix parent reflect">
 <joint name="${parent}_${suffix}_wheel_joint" type="continuous">
-	<parent link="${parent}_rotation_link"/>
+	<parent link="${parent}"/>
 	<child link="${parent}_${suffix}_wheel_link"/>
 	<origin rpy="0 0 0" xyz="0 0 0"/>
@@ -152,5 +152,5 @@
       </visual>
       <collision>
-        <!-- represent base collision with a simple rectangular model, positioned by base_size_z s.t. top
+        <!--represent base collision with a simple rectangular model, positioned by base_size_z s.t. top
 surface of the collision box matches the top surface of the PR2 base -->
         <origin xyz="0 0 ${0.051+talos_base_collision_size_z/2}" rpy="0 0 0" />

File: talos_navigation/talos_description/urdf/upper_arm_v0/talos_upper_arm_v1.urdf.xacro (robot description, xacro)
@@ -51,10 +51,10 @@
         <!-- TODO: Jordan end -->
         <!-- TODO: Someone? Not sure how these are done yet. -->
-	<collision>
+	<!-- <collision>
 		<origin xyz="0 0 0" rpy="0 0 0" />
 		<geometry>
-		  <!-- <mesh filename="package://pr2_description/meshes/upper_arm_v0/elbow_flex.stl" /> -->
+		  <mesh filename="package://pr2_description/meshes/upper_arm_v0/elbow_flex.stl" />
 		</geometry>
-	</collision>
+	</collision> -->
 	<visual>
 		<geometry>
@@ -101,11 +101,11 @@
         <!-- TODO: Jordan end -->
         <!-- TODO: Someone? Not sure how these are done yet. -->
-	<collision>
+	<!-- <collision>
 		<origin xyz="0 0 0" rpy="0 0 0" />
 		<geometry>
-		<!-- TODO: Add .stl file for proper collision matrix -->
-		  <!-- <mesh filename="package://pr2_description/meshes/upper_arm_v0/elbow_flex.stl" /> -->
+		TODO: Add .stl file for proper collision matrix
+		   <mesh filename="package://pr2_description/meshes/upper_arm_v0/elbow_flex.stl" />
 		</geometry>
-	</collision>
+	</collision> -->
 	<visual>
 		<geometry>

Commit message: Modified: base measurements

File: talos_navigation/talos_description/urdf/base_v0/talos_base.urdf.xacro (robot description, xacro)
@@ -43,7 +43,7 @@
 <property name="talos_base_collision_size_z" value="0" />
 <!-- TODO: Input proper values here -->
-<property name="talos_base_width" value="0" />
-<property name="talos_base_height" value="0" />
-<property name="talos_base_length" value="0" />
+<property name="talos_base_width" value="0.60" />
+<property name="talos_base_height" value="0.30" />
+<property name="talos_base_length" value="0.60" />
 <property name="talos_base_laser_x" value="0" />
 <property name="talos_base_laser_y" value="0" />

File: talos_navigation/talos_description/urdf/torso_v0/talos_torso.urdf.xacro (robot description, xacro)
@@ -22,4 +22,8 @@
 <property name="torso_safety_k_velocity" value="10"/>
 <property name="torso_mass" value="10" />
+<!-- END TODO -->
+<property name="talos_torso_width" value="0.4" />
+<property name="talos_torso_length" value="0.4" />
+<property name="talos_torso_height" value="1.0" />
 <!--                                               -->
 <!--                TORSO DEFINITION               -->
@@ -56,5 +60,5 @@
 	<!-- Temporary, because we will be using the .dae -->
 	<geometry>
-		<box size="0.4 0.4 1.0"/>
+		<box size="${talos_torso_length}  ${talos_torso_width} ${talos_torso_height}"/>
 	</geometry>
 	<material name="white">

Commit message: Fixed: Related kinks/bugs in urdf files Added: talos_common.urdf now represents approximately the robot's visual (Requires collisions, physics, transmissions, etc)

File: talos_navigation/talos_description/urdf/base_v0/talos_base.urdf.xacro (robot description, xacro)
@@ -52,9 +52,9 @@
 <!--                WHEEL DEFINITION               -->
 <!--                                               -->
-<xacro:macro name="talos_wheel" params="suffix parent reflect">
+<xacro:macro name="talos_wheel" params="suffix parent reflect_side reflect_back">
 <joint name="${parent}_${suffix}_wheel_joint" type="continuous">
 	<parent link="${parent}"/>
 	<child link="${parent}_${suffix}_wheel_link"/>
-	<origin rpy="0 0 0" xyz="0 0 0"/>
+	<origin rpy="0 1.57 0" xyz="${reflect_side*0.15} ${reflect_back*0.15} -0.15"/>
 	<axis xyz="0 1 0" />
        <limit effort="${max_wheel_effort}" velocity="${max_wheel_velocity}"/> <!-- alpha tested effort and velocity limits -->
@@ -72,5 +72,5 @@
         </geometry> -->
 		<origin rpy="0 0 0" xyz="0 0 0"/>
-		<material name="wheel_${suffix}">
+		<material name="black">
 			<color rgba="0 0 0 1"/>
 		</material>
@@ -170,8 +170,8 @@
     </xacro:hokuyo_lx30_laser_v0>
  <!-- Adding TALOS wheels to the base -->
-<xacro:talos_wheel suffix="fl" parent="talos_base" reflect="1" />
-<xacro:talos_wheel suffix="fr" parent="talos_base" reflect="-1" />
-<xacro:talos_wheel suffix="bl" parent="talos_base" reflect="1" />
-<xacro:talos_wheel suffix="br" parent="talos_base" reflect="-1" />
+<xacro:talos_wheel suffix="fl" parent="talos_base" reflect_side="1" reflect_back="1"/>
+<xacro:talos_wheel suffix="fr" parent="talos_base" reflect_side="-1" reflect_back="1"/>
+<xacro:talos_wheel suffix="bl" parent="talos_base" reflect_side="1" reflect_back="-1"/>
+<xacro:talos_wheel suffix="br" parent="talos_base" reflect_side="-1" reflect_back="-1"/>
 </xacro:macro>
 </robot>

File: talos_navigation/talos_description/urdf/talos_common.urdf (robot description, URDF)
Before this commit: robot talos, 9 links, 8 joints
Links:
- link talos_base: geometry visual box size=0.6 0.6 0.3
Joints:
- joint left_shoulder_joint: origin xyz=-0.25 -0.1 -0.39 rpy=0 0 1.57 -> xyz=0.25 0.1 0.39 rpy=0 0 1.57
- joint left_shoulder_to_upper_left_arm_joint: origin xyz=0 0.235 0 rpy=0 0 1.57 -> xyz=0 -0.235 0 rpy=1.57 0 0
- joint talos_base_bl_wheel_joint: origin xyz=0 0 0 rpy=0 0 0 -> xyz=0.15 -0.15 -0.15 rpy=0 1.57 0; parent talos_base_rotation_link -> talos_base
- joint talos_base_br_wheel_joint: origin xyz=0 0 0 rpy=0 0 0 -> xyz=-0.15 -0.15 -0.15 rpy=0 1.57 0; parent talos_base_rotation_link -> talos_base
- joint talos_base_fl_wheel_joint: origin xyz=0 0 0 rpy=0 0 0 -> xyz=0.15 0.15 -0.15 rpy=0 1.57 0; parent talos_base_rotation_link -> talos_base
- joint talos_base_fr_wheel_joint: origin xyz=0 0 0 rpy=0 0 0 -> xyz=-0.15 0.15 -0.15 rpy=0 1.57 0; parent talos_base_rotation_link -> talos_base
- joint torso_rotating_joint: origin xyz=0 0 0 rpy=0 0 0 -> xyz=0 0 0.5 rpy=0 0 0

File: talos_navigation/talos_description/urdf/talos_common.urdf.xacro (robot description, xacro)
@@ -24,5 +24,6 @@
 <property name="torso_offset_x" value="0" />
 <property name="torso_offset_y" value="0" />
-<property name="torso_offset_z" value="0" />
+<!-- VALUE: Torso height/2 + base height -->
+<property name="torso_offset_z" value="0.5" />
 <!--                                               -->
 <!--                 TALOS  DEFINITION             -->

File: talos_navigation/talos_description/urdf/torso_v0/talos_torso.urdf.xacro (robot description, xacro)
@@ -34,5 +34,5 @@
 	<parent link="${parent}"/>
 	<child link="${name}_link"/>
-	<origin rpy="0 0 0" xyz="0 0 0"/>
+        <xacro:insert_block name="origin" />
        <!-- TODO: Set appropriate values for these -->
 	<limit effort="${max_torso_effort}" velocity="${max_wheel_velocity}"/> <!-- alpha tested effort and velocity limits -->

File: talos_navigation/talos_description/urdf/upper_arm_v0/talos_upper_arm_v1.urdf.xacro (robot description, xacro)
@@ -37,5 +37,5 @@
   	<parent link="${parent}"/>
 	<child link="${side}_shoulder_link"/>
-	<origin rpy="0 0 1.57" xyz="-0.25 -0.1 -0.39"/>
+	<origin rpy="0 0 1.57" xyz="0.25 0.1 0.39"/>
 </joint>
 <link name="${side}_shoulder_link">
@@ -73,5 +73,5 @@
   	<parent link="${side}_shoulder_link"/>
 	<child link="${side}_upper_arm_link"/>
-	<origin rpy="0 0 1.57" xyz="0 0.235 0"/>
+	<origin rpy="1.57 0 0" xyz="0 -0.235 0"/>
 	<!-- Note: Code template taken from PR2_upper_arm.urdf for templating -->
 	<!-- Doc: axis of revolution -->

Commit message: Fixed bug where there was a double definition of the laser (so strange)

File: talos_navigation/talos_description/urdf/base_v0/talos_base.urdf.xacro (robot description, xacro)
@@ -49,4 +49,6 @@
 <property name="talos_base_laser_y" value="0" />
 <property name="talos_base_laser_z" value="0" />
+<!-- Half of wheel height + half of base height -->
+<property name="talos_base_z" value="${(wheel_radius/2)+(talos_base_height)/2}"/>
 <!--                                               -->
 <!--                WHEEL DEFINITION               -->
@@ -119,5 +121,5 @@
 			<box size="${talos_base_width} ${talos_base_length} ${talos_base_height}"/>
 		</geometry>
-		<origin rpy="0 0 0" xyz="0 0 0"/>
+		<origin rpy="0 0 0" xyz="0 0 ${talos_base_z}"/>
               <!-- TODO: Replace with .stl file -->
 		<material name="white">
@@ -165,8 +167,9 @@
       <parent link="${name}_base_footprint"/>
     </joint>
-  <!-- base laser -->
+<!-- I'm not sure how this got added in.. but what the fuck?
     <xacro:hokuyo_lx30_laser_v0 name="${name}_base_laser" parent="talos_base" ros_topic="base_scan" update_rate="20" min_angle="-2.2689" max_angle="2.2689" >
       <origin xyz="${talos_base_laser_x} ${talos_base_laser_y} ${talos_base_laser_z}" rpy="0 0 0" />
     </xacro:hokuyo_lx30_laser_v0>
+ It should've been in the tilting laser file.. -->
  <!-- Adding TALOS wheels to the base -->
 <xacro:talos_wheel suffix="fl" parent="talos_base" reflect_side="1" reflect_back="1"/>

Commit message: Fixed: bugs with the TF tree

File: talos_navigation/talos_description/urdf/base_v0/talos_base.urdf.xacro (robot description, xacro)
@@ -107,5 +107,5 @@
 <!--                       Base Definition                 -->
 <xacro:macro name="talos_base" params="name">
-<link name="talos_base">
+<link name="talos_base_link">
 	<!-- TODO: Jordan to put proper values for the xml below
 	<inertial>
@@ -164,5 +164,5 @@
     <joint name="${name}_base_footprint_joint" type="fixed">
       <origin xyz="0 0 0.051" rpy="0 0 0" />
-      <child link="talos_base" />
+      <child link="talos_base_link" />
       <parent link="${name}_base_footprint"/>
     </joint>
@@ -173,8 +173,8 @@
  It should've been in the tilting laser file.. -->
  <!-- Adding TALOS wheels to the base -->
-<xacro:talos_wheel suffix="fl" parent="talos_base" reflect_side="1" reflect_back="1"/>
-<xacro:talos_wheel suffix="fr" parent="talos_base" reflect_side="-1" reflect_back="1"/>
-<xacro:talos_wheel suffix="bl" parent="talos_base" reflect_side="1" reflect_back="-1"/>
-<xacro:talos_wheel suffix="br" parent="talos_base" reflect_side="-1" reflect_back="-1"/>
+<xacro:talos_wheel suffix="fl" parent="talos_base_link" reflect_side="1" reflect_back="1"/>
+<xacro:talos_wheel suffix="fr" parent="talos_base_link" reflect_side="-1" reflect_back="1"/>
+<xacro:talos_wheel suffix="bl" parent="talos_base_link" reflect_side="1" reflect_back="-1"/>
+<xacro:talos_wheel suffix="br" parent="talos_base_link" reflect_side="-1" reflect_back="-1"/>
 </xacro:macro>
 </robot>

File: talos_navigation/talos_description/urdf/talos_common.urdf (robot description, URDF)
Before this commit: robot talos, 14 links, 13 joints
Joints:
- removed joint talos_base_link_hack

File: talos_navigation/talos_description/urdf/tilting_laser_v0/talos_tilting_laser.urdf.xacro (robot description, xacro)
@@ -15,4 +15,5 @@
 <property name="talos_base_laser_z" value="0.3" />
 <property name="M_PI" value="3.1415926535897931"/>
+<!-- No longer need small hack, DEPRECATED
 Small hack to get around the fact that hokuyo xacro adds a _link to the parent name
 <link name="talos_base_link">
@@ -23,5 +24,5 @@
       </geometry>
     </visual>
-</link>
+</link>  -->
 <!--
 <joint name="talos_base_link_hack" type="fixed">
