Commit message: Added: things

File: talos_navigation/talos_description/urdf/base_v0/talos_base.urdf.xacro (robot description, xacro)
@@ -121,5 +121,5 @@
 			<box size="${talos_base_width} ${talos_base_length} ${talos_base_height}"/>
 		</geometry>
-		<origin rpy="0 0 0" xyz="0 0 ${talos_base_z}"/>
+		<origin rpy="0 0 0" xyz="0 0 0"/>
               <!-- TODO: Replace with .stl file -->
 		<material name="white">
@@ -163,5 +163,5 @@
     </link>
     <joint name="${name}_base_footprint_joint" type="fixed">
-      <origin xyz="0 0 0.051" rpy="0 0 0" />
+      <origin xyz="0 0 ${talos_base_z}" rpy="0 0 0" />
       <child link="talos_base_link" />
       <parent link="${name}_base_footprint"/>

File: talos_navigation/talos_description/urdf/talos_common.urdf (robot description, URDF)
Before this commit: robot talos, 14 links, 12 joints
Links:
- removed link talos_base
- removed link talos_base_bl_wheel_link
- removed link talos_base_br_wheel_link
- removed link talos_base_fl_wheel_link
- removed link talos_base_fr_wheel_link
- added link talos_base_link_bl_wheel_link; visual cylinder length=0.01 radius=0.0761
- added link talos_base_link_br_wheel_link; visual cylinder length=0.01 radius=0.0761
- added link talos_base_link_fl_wheel_link; visual cylinder length=0.01 radius=0.0761
- added link talos_base_link_fr_wheel_link; visual cylinder length=0.01 radius=0.0761
- link talos_base_link: geometry visual box size=0.6 0.6 0.3
Joints:
- removed joint talos_base_bl_wheel_joint
- removed joint talos_base_br_wheel_joint
- removed joint talos_base_fl_wheel_joint
- removed joint talos_base_fr_wheel_joint
- added joint talos_base_link_bl_wheel_joint: type continuous, parent talos_base_link, child talos_base_link_bl_wheel_link, origin xyz=0.15 -0.15 -0.15 rpy=0 1.57 0, axis 0 1 0, limit effort=7 velocity=15
- added joint talos_base_link_br_wheel_joint: type continuous, parent talos_base_link, child talos_base_link_br_wheel_link, origin xyz=-0.15 -0.15 -0.15 rpy=0 1.57 0, axis 0 1 0, limit effort=7 velocity=15
- added joint talos_base_link_fl_wheel_joint: type continuous, parent talos_base_link, child talos_base_link_fl_wheel_link, origin xyz=0.15 0.15 -0.15 rpy=0 1.57 0, axis 0 1 0, limit effort=7 velocity=15
- added joint talos_base_link_fr_wheel_joint: type continuous, parent talos_base_link, child talos_base_link_fr_wheel_link, origin xyz=-0.15 0.15 -0.15 rpy=0 1.57 0, axis 0 1 0, limit effort=7 velocity=15
- joint talos_base_footprint_joint: child talos_base -> talos_base_link; origin xyz=0 0 0.051 rpy=0 0 0 -> xyz=0 0 0.18805 rpy=0 0 0
- joint torso_rotating_joint: parent talos_base -> talos_base_link
